File: Schematic/prize_delivery.brd (EAGLE design)
At the start: 100.1 x 43.2 mm, 13 parts, among them Q1 IRL540

Commit message: Modified schematic
Parts:
- removed 180°, 360°, START: MOMENTARY-SWITCH-SPST-PTH-6.0MM, SparkFun-Switches:TACTILE_SWITCH_PTH_6.0MM
- removed JP1: Start, pinhead:1X02
- added JP4: (no value), adafruit:1X06
Connections:
- removed net 5V: W1.JP2.8
- net 0: now also JP4.1; no longer 180°.3, 360°.3, JP1.1, START.3
- net N$3: now also W1.JP2.8
- net N$4: now also JP4.3; no longer 180°.1
- net N$5: now also JP4.4; no longer 360°.1
- net N$9: now also JP4.2; no longer JP1.2, START.1
Routing:
- net 0: track 147.1 -> 104.3 mm
- net N$3: track 21.9 -> 5.39 mm
- net N$9: track 94.6 -> 88.6 mm
Changed lines of the file:
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@@
 </autorouter>
 <elements>
-<element name="START" library="SparkFun-Switches" library_urn="urn:adsk.eagle:library:535" package="TACTILE_SWITCH_PTH_6.0MM" package3d_urn="urn:adsk.eagle:package:40163/1" value="MOMENTARY-SWITCH-SPST-PTH-6.0MM" x="15.24" y="7.62" smashed="yes">
-<attribute name="NAME" x="15.24" y="10.922" size="0.6096" layer="25" font="vector" ratio="20" align="bottom-center"/>
-<attribute name="PROD_ID" value=" SWCH-08441" x="49.53" y="-31.75" size="1.778" layer="27" display="off"/>
-<attribute name="SF_SKU" value="COM-00097" x="49.53" y="-31.75" size="1.778" layer="27" display="off"/>
-</element>
 <element name="D1" library="adafruit" library_urn="urn:adsk.eagle:library:420" package="DO41-10" package3d_urn="urn:adsk.eagle:package:6240344/1" value="1N4004" x="22.86" y="27.94" smashed="yes" rot="R90">
 <attribute name="NAME" x="21.209" y="25.908" size="1.27" layer="25" ratio="10" rot="R90"/>
@@
 <attribute name="VALUE" x="25.6794" y="15.875" size="1.27" layer="27" ratio="10"/>
 </element>
-<element name="180°" library="SparkFun-Switches" library_urn="urn:adsk.eagle:library:535" package="TACTILE_SWITCH_PTH_6.0MM" package3d_urn="urn:adsk.eagle:package:40163/1" value="MOMENTARY-SWITCH-SPST-PTH-6.0MM" x="29.21" y="7.62" smashed="yes">
-<attribute name="NAME" x="29.21" y="10.922" size="0.6096" layer="25" font="vector" ratio="20" align="bottom-center"/>
-<attribute name="PROD_ID" value=" SWCH-08441" x="50.8" y="-41.91" size="1.778" layer="27" display="off"/>
-<attribute name="SF_SKU" value="COM-00097" x="50.8" y="-41.91" size="1.778" layer="27" display="off"/>
-</element>
-<element name="360°" library="SparkFun-Switches" library_urn="urn:adsk.eagle:library:535" package="TACTILE_SWITCH_PTH_6.0MM" package3d_urn="urn:adsk.eagle:package:40163/1" value="MOMENTARY-SWITCH-SPST-PTH-6.0MM" x="44.45" y="7.62" smashed="yes">
-<attribute name="NAME" x="44.45" y="10.922" size="0.6096" layer="25" font="vector" ratio="20" align="bottom-center"/>
-<attribute name="PROD_ID" value=" SWCH-08441" x="83.82" y="-41.91" size="1.778" layer="27" display="off"/>
-<attribute name="SF_SKU" value="COM-00097" x="83.82" y="-41.91" size="1.778" layer="27" display="off"/>
-</element>
 <element name="W1" library="diy-modules" package="WEMOS-D1-MINI" value="WEMOS-D1-MINI" x="82.55" y="20.32" smashed="yes" rot="R90"/>
 <element name="R2" library="adafruit" library_urn="urn:adsk.eagle:library:420" package="0207/10" package3d_urn="urn:adsk.eagle:package:6240597/1" value="470" x="53.34" y="24.13" smashed="yes">
@@
 <attribute name="VALUE" x="9.525" y="22.86" size="1.27" layer="27" rot="R90"/>
 </element>
-<element name="JP1" library="pinhead" library_urn="urn:adsk.eagle:library:325" package="1X02" package3d_urn="urn:adsk.eagle:package:22435/2" value="Start" x="6.35" y="19.05" smashed="yes" rot="R90">
-<attribute name="NAME" x="4.5212" y="16.4338" size="1.27" layer="25" ratio="10" rot="R90"/>
-<attribute name="POPULARITY" value="98" x="6.35" y="19.05" size="1.778" layer="27" rot="R90" display="off"/>
-<attribute name="VALUE" x="9.525" y="16.51" size="1.27" layer="27" rot="R90"/>
+<element name="JP4" library="adafruit" package="1X06" value="" x="6.35" y="13.97" smashed="yes" rot="R90">
+<attribute name="NAME" x="4.5212" y="6.2738" size="1.27" layer="25" ratio="10" rot="R90"/>
+<attribute name="VALUE" x="9.525" y="6.35" size="1.27" layer="27" rot="R90"/>
 </element>
 </elements>
@@
 </signal>
 <signal name="0">
-<contactref element="180°" pad="3"/>
-<contactref element="360°" pad="3"/>
 <contactref element="Q1" pad="3"/>
 <contactref element="W1" pad="JP2.7"/>
-<contactref element="START" pad="3"/>
 <contactref element="R1" pad="2"/>
 <contactref element="R4" pad="1"/>
-<contactref element="JP2" pad="1"/>
-<contactref element="JP1" pad="1"/>
-<wire x1="8.255" y1="19.685" x2="6.35" y2="17.78" width="0.1524" layer="16"/>
-<wire x1="8.255" y1="22.225" x2="8.255" y2="19.685" width="0.1524" layer="16"/>
-<wire x1="6.35" y1="24.13" x2="8.255" y2="22.225" width="0.1524" layer="16"/>
 <wire x1="22.86" y1="5.3975" x2="22.86" y2="6.6675" width="0.1524" layer="1"/>
 <wire x1="22.86" y1="6.6675" x2="22.86" y2="16.51" width="0.1524" layer="1"/>
 <wire x1="25.7175" y1="5.3975" x2="22.86" y2="5.3975" width="0.1524" layer="1"/>
-<wire x1="25.7175" y1="5.3975" x2="25.9588" y2="5.3594" width="0.1524" layer="1"/>
 <wire x1="13.335" y1="6.6675" x2="12.065" y2="5.3975" width="0.1524" layer="1"/>
 <wire x1="22.86" y1="6.6675" x2="13.335" y2="6.6675" width="0.1524" layer="1"/>
-<wire x1="12.065" y1="5.3975" x2="11.9888" y2="5.3594" width="0.1524" layer="1"/>
-<wire x1="6.35" y1="5.3975" x2="6.35" y2="17.78" width="0.1524" layer="1"/>
-<wire x1="11.7475" y1="5.3975" x2="6.35" y2="5.3975" width="0.1524" layer="1"/>
-<wire x1="11.7475" y1="5.3975" x2="11.9888" y2="5.3594" width="0.1524" layer="1"/>
 <wire x1="74.295" y1="17.78" x2="88.265" y2="31.75" width="0.1524" layer="1"/>
 <wire x1="49.53" y1="17.78" x2="74.295" y2="17.78" width="0.1524" layer="1"/>
@@
 <wire x1="46.99" y1="11.1125" x2="41.275" y2="5.3975" width="0.1524" layer="16"/>
 <wire x1="46.99" y1="16.51" x2="46.99" y2="11.1125" width="0.1524" layer="16"/>
-<wire x1="41.275" y1="5.3975" x2="41.1988" y2="5.3594" width="0.1524" layer="16"/>
-<wire x1="26.9875" y1="4.1275" x2="26.035" y2="5.08" width="0.1524" layer="1"/>
-<wire x1="40.005" y1="4.1275" x2="26.9875" y2="4.1275" width="0.1524" layer="1"/>
-<wire x1="40.9575" y1="5.08" x2="40.005" y2="4.1275" width="0.1524" layer="1"/>
-<wire x1="26.035" y1="5.08" x2="25.9588" y2="5.3594" width="0.1524" layer="1"/>
-<wire x1="40.9575" y1="5.08" x2="41.1988" y2="5.3594" width="0.1524" layer="1"/>
+<contactref element="JP4" pad="1"/>
+<contactref element="JP2" pad="1"/>
+<wire x1="25.7175" y1="5.3975" x2="41.275" y2="5.3975" width="0" layer="19" extent="1-16"/>
+<wire x1="6.35" y1="7.62" x2="12.065" y2="5.3975" width="0" layer="19" extent="1-1"/>
+<wire x1="6.35" y1="24.13" x2="22.86" y2="16.51" width="0" layer="19" extent="1-1"/>
 </signal>
 <signal name="N$1">
@@
 <signal name="N$3">
 <contactref element="JP3" pad="1"/>
+<contactref element="D1" pad="C"/>
+<wire x1="19.05" y1="26.67" x2="22.86" y2="22.86" width="0.1524" layer="1"/>
 <contactref element="JP2" pad="2"/>
-<contactref element="D1" pad="C"/>
-<wire x1="6.35" y1="30.48" x2="6.35" y2="26.67" width="0.1524" layer="1"/>
-<wire x1="19.05" y1="26.67" x2="22.86" y2="22.86" width="0.1524" layer="1"/>
-<wire x1="6.35" y1="26.67" x2="19.05" y2="26.67" width="0.1524" layer="1"/>
+<contactref element="W1" pad="JP2.8"/>
+<wire x1="22.86" y1="22.86" x2="90.805" y2="31.75" width="0" layer="19" extent="1-1"/>
+<wire x1="6.35" y1="26.67" x2="19.05" y2="26.67" width="0" layer="19" extent="1-1"/>
+<wire x1="6.35" y1="30.48" x2="6.35" y2="26.67" width="0" layer="19" extent="1-1"/>
 </signal>
 <signal name="N$4">
-<contactref element="180°" pad="1"/>
 <contactref element="W1" pad="JP2.4"/>
 <wire x1="76.835" y1="35.56" x2="80.645" y2="31.75" width="0.1524" layer="16"/>
 <wire x1="26.035" y1="35.56" x2="76.835" y2="35.56" width="0.1524" layer="16"/>
 <wire x1="26.035" y1="10.16" x2="26.035" y2="35.56" width="0.1524" layer="16"/>
-<wire x1="26.035" y1="10.16" x2="25.9588" y2="9.8806" width="0.1524" layer="16"/>
+<contactref element="JP4" pad="3"/>
+<wire x1="6.35" y1="12.7" x2="26.035" y2="10.16" width="0" layer="19" extent="16-16"/>
 </signal>
 <signal name="N$5">
 <contactref element="W1" pad="JP2.3"/>
-<contactref element="360°" pad="1"/>
 <wire x1="50.4825" y1="4.1275" x2="78.105" y2="31.75" width="0.1524" layer="16"/>
 <wire x1="40.005" y1="4.1275" x2="50.4825" y2="4.1275" width="0.1524" layer="16"/>
 <wire x1="40.005" y1="8.89" x2="40.005" y2="4.1275" width="0.1524" layer="16"/>
 <wire x1="40.9575" y1="9.8425" x2="40.005" y2="8.89" width="0.1524" layer="16"/>
-<wire x1="40.9575" y1="9.8425" x2="41.1988" y2="9.8806" width="0.1524" layer="16"/>
+<contactref element="JP4" pad="4"/>
+<wire x1="6.35" y1="15.24" x2="40.9575" y2="9.8425" width="0" layer="19" extent="16-16"/>
 </signal>
 <signal name="N$7">
@@
 </signal>
 <signal name="N$9">
-<contactref element="START" pad="1"/>
 <contactref element="W1" pad="JP2.6"/>
-<contactref element="JP1" pad="2"/>
 <wire x1="74.295" y1="20.32" x2="85.725" y2="31.75" width="0.1524" layer="1"/>
-<wire x1="6.35" y1="20.32" x2="12.065" y2="20.32" width="0.1524" layer="1"/>
 <wire x1="12.065" y1="20.32" x2="74.295" y2="20.32" width="0.1524" layer="1"/>
 <wire x1="12.065" y1="20.32" x2="12.065" y2="10.16" width="0.1524" layer="1"/>
-<wire x1="12.065" y1="10.16" x2="11.9888" y2="9.8806" width="0.1524" layer="1"/>
+<contactref element="JP4" pad="2"/>
+<wire x1="6.35" y1="10.16" x2="12.065" y2="10.16" width="0" layer="19" extent="1-1"/>
 </signal>
 <signal name="N$6">
@@
 <wire x1="34.29" y1="24.13" x2="48.26" y2="24.13" width="0.1524" layer="1"/>
 </signal>
-<signal name="5V">
-<contactref element="W1" pad="JP2.8"/>
-</signal>
 </signals>

Commit message: Update PCB
Parts:
- removed JP3: Motor, pinhead:1X02
- removed JP4: (no value), adafruit:1X06
- removed Q1: IRL540, adafruit:TO220V
- added JP1: (no value), pinhead:1X04
- added Q2: RFP30N06LE, RFP30N06LE:TRANS_RFP30N06LE
- JP2: value 5Vin -> (none); device pinhead:1X02 -> pinhead:1X04
- moved D1 18.9 mm to (35.6, 14.0), turned to 0 degrees
- moved JP2 13.0 mm to (19.1, 27.9)
- moved R4 8.52 mm to (35.6, 20.3)
- moved R2 3.81 mm to (53.3, 20.3)
- moved R1 2.54 mm to (53.3, 14.0)
Connections:
- removed net N$14: Q1.1, R2.1, R4.2
- new net N$8: Q2.1, R2.1, R4.2
- net 0: now also JP1.1, Q2.3; no longer JP4.1, Q1.3
- net N$2: now also JP1.4, Q2.2; no longer JP3.2, Q1.2
- net N$3: now also JP1.2, JP1.3; no longer JP2.2, JP3.1
- net N$4: now also JP2.3; no longer JP4.3
- net N$5: now also JP2.4; no longer JP4.4
- net N$9: now also JP2.2; no longer JP4.2
Routing:
- net N$3: track 5.39 -> 82.9 mm
- net N$14: track 22.1 -> 0.00 mm
- net N$4: track 81.6 -> 62.7 mm
- net N$8: track 0.00 -> 16.5 mm
- net N$2: track 30.6 -> 40.0 mm
- net N$5: track 55.7 -> 62.1 mm
- net 0: track 104.3 -> 108.4 mm
- net N$7: track 8.89 -> 6.41 mm
- net N$1: track 27.9 -> 29.5 mm
- net N$9: track 88.6 -> 87.8 mm
Other:
- board size 100.1 x 43.2 mm -> 88.6 x 40.6 mm
- board text added: "+5V"
- board text added: "180°"
- board text added: "360°"
- board text added: "Gnd"
- board text added: "M+"
- board text added: "M-"
- board text added: "Start"
