File: PrizeDelivery/Schematic/prize_delivery.brd (EAGLE design)
At the start: 93.7 x 38.1 mm, 13 parts, among them Q1 IRL540

Commit message: Added images folder
Parts:
- removed 180°: MOMENTARY-SWITCH-SPST-PTH-6.0MM, SparkFun-Switches:TACTILE_SWITCH_PTH_6.0MM
- added LED2, LED3, LED4, LED6, LED7: (no value), adafruit:LED5MM
- added R3, R5, R6, R8, R9: 1K, adafruit:0207/10
- renumbered LED1 to STATUS
Connections:
- new net N$11: LED6.K, R8.1
- new net N$12: LED7.K, R9.1
- new net N$15: LED2.A, W1.JP1.3
- new net N$16: LED3.A, W1.JP1.5
- new net N$17: LED4.A, W1.JP1.6
- new net N$18: LED7.A, W1.JP2.1
- new net N$19: LED6.A, W1.JP2.2
- new net N$20: STATUS.A, W1.JP1.4
- new net N$8: LED4.K, R6.1
- net 0: now also R3.2, R5.2, R6.2, R8.2, R9.2; no longer 180°.3
- net N$1: now also LED2.K, R3.1; no longer R2.2, W1.JP2.5
- net N$4: now also LED3.K, R5.1; no longer 180°.1, W1.JP2.4
- net N$5: now also W1.JP2.4; no longer W1.JP2.3
- net N$6: now also R2.2, W1.JP2.3; no longer STATUS.A, W1.JP1.7
Routing:
- net N$4: track 60.3 -> 0.00 mm
- net N$1: track 40.0 -> 0.00 mm
- net N$6: track 34.5 -> 0.00 mm
- net N$9: track 90.6 -> 89.4 mm
- net N$5: track 73.0 -> 71.8 mm

Commit message: Not sure
Parts:
- removed LED2, LED3, LED4, LED6, LED7, STATUS: (no value), adafruit:LED5MM
- removed R1, R3, R5, R6, R8, R9: 1K, adafruit:0207/10
- added J2: (no value), Wurth_Elektronik_Electromechanic_Terminal_Blocks_Connectors_rev19b:691136710008
Connections:
- removed net N$1: LED2.K, R3.1
- removed net N$11: LED6.K, R8.1
- removed net N$12: LED7.K, R9.1
- removed net N$4: LED3.K, R5.1
- removed net N$7: R1.1, STATUS.K
- removed net N$8: LED4.K, R6.1
- net 0: now also J2.1; no longer R1.2, R3.2, R5.2, R6.2, R8.2, R9.2
- net N$15: now also J2.4; no longer LED2.A
- net N$16: now also J2.5; no longer LED3.A
- net N$17: now also J2.6; no longer LED4.A
- net N$18: now also J2.8; no longer LED7.A
- net N$19: now also J2.7; no longer LED6.A
- net N$20: now also J2.3; no longer STATUS.A
- net N$9: now also J2.2
Routing:
- net 0: track 138.6 -> 124.4 mm
- net N$7: track 6.88 -> 0.00 mm
